Commit message: 追加

File: work/src/magician_rl/magician_suction_optimized.urdf (robot description, URDF)
Before this commit: robot magician, 8 links, 7 joints
Links:
- link magician_base_link: geometry collision box size=0.2 0.2 0.05; visual mesh filename=meshes/dae/magicianBase.dae
- link magician_link_1: geometry collision cylinder length=0.1 radius=0.05; visual mesh filename=meshes/dae/magicianLink1.dae
- link magician_link_2: geometry collision box size=0.05 0.05 0.14; visual mesh filename=meshes/dae/magicianLink2.dae
- link magician_link_3: geometry collision box size=0.14 0.05 0.05; visual mesh filename=meshes/dae/magicianLink3.dae
- link magician_link_4: geometry collision box size=0.06 0.04 0.04; visual mesh filename=meshes/collision/end_tools/suction_cup_collision_part1.dae
- link magician_link_gripper_core: geometry collision cylinder length=0.04 radius=0.01; visual mesh filename=meshes/collision/end_tools/suction_cup_collision_part2.dae
